File: RNS_Board.brd (EAGLE design)
At the start: 67.3 x 65.7 mm, 6 parts

Commit message: Add files via upload
Connections:
- net 3.3V@2: now also JP6.1
- net 5V: no longer JP6.1
Routing:
- net 5V: track 126.3 -> 69.2 mm
- net 3.3V@2: track 0.00 -> 18.8 mm
- net GND@2: track 17.0 -> 30.8 mm
- net GND@1: track 102.1 -> 108.4 mm
- net PB_3: track 12.0 -> 13.2 mm
Other:
- board size 67.3 x 65.7 mm -> 71.1 x 65.7 mm
Changed lines of the file:
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@@
 <layer number="16" name="Bottom" color="1" fill="1" visible="yes" active="yes"/>
 <layer number="17" name="Pads" color="2" fill="1" visible="yes" active="yes"/>
-<layer number="18" name="Vias" color="2" fill="1" visible="yes" active="yes"/>
-<layer number="19" name="Unrouted" color="6" fill="1" visible="yes" active="yes"/>
+<layer number="18" name="Vias" color="2" fill="1" visible="no" active="yes"/>
+<layer number="19" name="Unrouted" color="6" fill="1" visible="no" active="yes"/>
 <layer number="20" name="Dimension" color="24" fill="1" visible="yes" active="yes"/>
-<layer number="21" name="tPlace" color="7" fill="1" visible="yes" active="yes"/>
-<layer number="22" name="bPlace" color="7" fill="1" visible="yes" active="yes"/>
-<layer number="23" name="tOrigins" color="15" fill="1" visible="yes" active="yes"/>
-<layer number="24" name="bOrigins" color="15" fill="1" visible="yes" active="yes"/>
-<layer number="25" name="tNames" color="7" fill="1" visible="yes" active="yes"/>
-<layer number="26" name="bNames" color="7" fill="1" visible="yes" active="yes"/>
-<layer number="27" name="tValues" color="7" fill="1" visible="yes" active="yes"/>
-<layer number="28" name="bValues" color="7" fill="1" visible="yes" active="yes"/>
+<layer number="21" name="tPlace" color="7" fill="1" visible="no" active="yes"/>
+<layer number="22" name="bPlace" color="7" fill="1" visible="no" active="yes"/>
+<layer number="23" name="tOrigins" color="15" fill="1" visible="no" active="yes"/>
+<layer number="24" name="bOrigins" color="15" fill="1" visible="no" active="yes"/>
+<layer number="25" name="tNames" color="7" fill="1" visible="no" active="yes"/>
+<layer number="26" name="bNames" color="7" fill="1" visible="no" active="yes"/>
+<layer number="27" name="tValues" color="7" fill="1" visible="no" active="yes"/>
+<layer number="28" name="bValues" color="7" fill="1" visible="no" active="yes"/>
 <layer number="29" name="tStop" color="7" fill="3" visible="no" active="yes"/>
 <layer number="30" name="bStop" color="7" fill="6" visible="no" active="yes"/>
@@
 <board>
 <plain>
-<wire x1="-3.81" y1="0" x2="63.48" y2="0" width="0" layer="20"/>
+<wire x1="-7.62" y1="0" x2="63.48" y2="0" width="0" layer="20"/>
 <wire x1="63.48" y1="0" x2="63.48" y2="65.71" width="0" layer="20"/>
-<wire x1="63.48" y1="65.71" x2="-3.81" y2="65.71" width="0" layer="20"/>
-<wire x1="-3.81" y1="65.71" x2="-3.81" y2="0" width="0" layer="20"/>
+<wire x1="63.48" y1="65.71" x2="-7.62" y2="65.71" width="0" layer="20"/>
+<wire x1="-7.62" y1="65.71" x2="-7.62" y2="0" width="0" layer="20"/>
 </plain>
 <attributes>
@@
 <elements>
 <element name="JP1" library="MIA_LIBRARY-2-2-2" package="1X02" package3d_urn="urn:adsk.eagle:package:22435/2" value="" x="3.81" y="12.7" smashed="yes" rot="R90" grouprefs="RNS">
-<attribute name="NAME" x="1.9812" y="10.0838" size="1.27" layer="25" ratio="10" rot="R90"/>
 <attribute name="POPULARITY" value="98" x="36.83" y="38.1" size="1.778" layer="27" rot="R90" display="off"/>
 <attribute name="VALUE" x="6.985" y="10.16" size="1.27" layer="27" rot="R90"/>
 </element>
 <element name="JP2" library="MIA_LIBRARY-2-2-2" package="1X03" package3d_urn="urn:adsk.eagle:package:22458/2" value="" x="3.81" y="52.07" smashed="yes" rot="R83.7" grouprefs="RNS">
-<attribute name="NAME" x="0.29579375" y="49.67795" size="1.27" layer="25" ratio="10" rot="R83.7"/>
 <attribute name="POPULARITY" value="92" x="38.581665625" y="66.119196875" size="1.778" layer="27" rot="R83.7" display="off"/>
 <attribute name="VALUE" x="6.5477375" y="47.9346" size="1.27" layer="27" rot="R83.7"/>
 </element>
 <element name="JP4" library="MIA_LIBRARY-2-2-2" package="1X04" package3d_urn="urn:adsk.eagle:package:22407/2" value="" x="5.08" y="30.48" smashed="yes" rot="R90" grouprefs="RNS">
-<attribute name="NAME" x="0.7112" y="26.5938" size="1.27" layer="25" ratio="10" rot="R90"/>
 <attribute name="POPULARITY" value="91" x="31.75" y="49.53" size="1.778" layer="27" rot="R90" display="off"/>
 <attribute name="VALUE" x="8.255" y="25.4" size="1.27" layer="27" rot="R90"/>
@@
 </element>
 <element name="JP6" library="MIA_LIBRARY-2-2-2" package="1X04" package3d_urn="urn:adsk.eagle:package:22407/2" value="" x="49.53" y="53.34" smashed="yes" rot="R270" grouprefs="RNS">
-<attribute name="NAME" x="51.3588" y="58.4962" size="1.27" layer="25" ratio="10" rot="R270"/>
 <attribute name="POPULARITY" value="91" x="22.86" y="11.43" size="1.778" layer="27" rot="R270" display="off"/>
 <attribute name="VALUE" x="46.355" y="58.42" size="1.27" layer="27" rot="R270"/>
@@
 <contactref element="U$1" pad="PB_3"/>
 <contactref element="JP4" pad="4"/>
-<wire x1="17.78" y1="33.02" x2="12.7" y2="33.02" width="1.016" layer="16" grouprefs="RNS"/>
-<wire x1="12.7" y1="33.02" x2="11.43" y2="34.29" width="1.016" layer="16" grouprefs="RNS"/>
-<wire x1="11.43" y1="34.29" x2="6.35" y2="34.29" width="1.016" layer="16" grouprefs="RNS"/>
-<wire x1="6.35" y1="34.29" x2="5.08" y2="34.29" width="0" layer="19" extent="16-16"/>
+<wire x1="17.78" y1="33.02" x2="12.7" y2="33.02" width="0.8128" layer="16"/>
+<wire x1="12.7" y1="33.02" x2="11.43" y2="34.29" width="0.8128" layer="16"/>
+<wire x1="11.43" y1="34.29" x2="5.08" y2="34.29" width="0.8128" layer="16"/>
 </signal>
 <signal name="PB_4">
@@
 <contactref element="JP4" pad="1"/>
 <contactref element="JP1" pad="2"/>
-<contactref element="JP6" pad="1"/>
 <contactref element="JP5" pad="3"/>
 <wire x1="17.78" y1="15.24" x2="7.62" y2="15.24" width="1.016" layer="16" grouprefs="RNS"/>
@@
 <wire x1="5.08" y1="26.67" x2="5.08" y2="17.78" width="1.016" layer="16" grouprefs="RNS"/>
 <wire x1="5.08" y1="17.78" x2="7.62" y2="15.24" width="1.016" layer="16" grouprefs="RNS"/>
-<wire x1="49.53" y1="20.32" x2="48.4124" y2="19.2024" width="1.016" layer="16" grouprefs="RNS"/>
 <wire x1="34.28915625" y1="8.7956" x2="31.75084375" y2="8.7956" width="1.016" layer="16" grouprefs="RNS"/>
 <wire x1="31.75084375" y1="8.7956" x2="31.65644375" y2="8.89" width="1.016" layer="16" grouprefs="RNS"/>
 <wire x1="31.65644375" y1="8.89" x2="24.13" y2="8.89" width="1.016" layer="16" grouprefs="RNS"/>
-<wire x1="48.4124" y1="19.2024" x2="44.69595625" y2="19.2024" width="1.016" layer="16" grouprefs="RNS"/>
 <wire x1="44.69595625" y1="19.2024" x2="34.28915625" y2="8.7956" width="1.016" layer="16" grouprefs="RNS"/>
 <wire x1="24.13" y1="8.89" x2="22.86" y2="10.16" width="1.016" layer="16" grouprefs="RNS"/>
 <wire x1="22.86" y1="10.16" x2="22.86" y2="15.24" width="1.016" layer="16" grouprefs="RNS"/>
 <wire x1="22.86" y1="15.24" x2="17.78" y2="15.24" width="1.016" layer="16" grouprefs="RNS"/>
-<wire x1="49.53" y1="57.15" x2="59.69" y2="57.15" width="1.016" layer="16" grouprefs="RNS"/>
-<wire x1="59.69" y1="57.15" x2="59.69" y2="20.32" width="1.016" layer="16" grouprefs="RNS"/>
-<wire x1="59.69" y1="20.32" x2="49.53" y2="20.32" width="1.016" layer="16" grouprefs="RNS"/>
+<wire x1="49.53" y1="20.32" x2="45.72" y2="20.32" width="0.8128" layer="16"/>
+<wire x1="45.72" y1="20.32" x2="44.69595625" y2="19.29595625" width="0.8128" layer="16"/>
+<wire x1="44.69595625" y1="19.29595625" x2="44.69595625" y2="19.2024" width="0.8128" layer="16"/>
 </signal>
 <signal name="GND@1">
@@
 <wire x1="16.51084375" y1="11.5244" x2="16.41644375" y2="11.43" width="1.016" layer="16" grouprefs="RNS"/>
 <wire x1="16.41644375" y1="11.43" x2="5.08" y2="11.43" width="1.016" layer="16" grouprefs="RNS"/>
-<wire x1="5.08" y1="29.21" x2="1.524" y2="29.21" width="1.016" layer="16" grouprefs="RNS"/>
-<wire x1="1.524" y1="7.62" x2="1.524" y2="29.21" width="1.016" layer="16" grouprefs="RNS"/>
 <wire x1="3.81" y1="11.43" x2="3.81" y2="6.35" width="1.016" layer="16" grouprefs="RNS"/>
-<wire x1="3.81" y1="6.35" x2="2.794" y2="6.35" width="1.016" layer="16" grouprefs="RNS"/>
-<wire x1="2.794" y1="6.35" x2="1.524" y2="7.62" width="1.016" layer="16" grouprefs="RNS"/>
+<wire x1="2.794" y1="6.35" x2="3.81" y2="6.35" width="1.016" layer="16" grouprefs="RNS"/>
 <wire x1="49.53" y1="17.78" x2="34.29" y2="2.54" width="1.016" layer="16" grouprefs="RNS"/>
 <wire x1="34.29" y1="2.54" x2="3.81" y2="2.54" width="1.016" layer="16" grouprefs="RNS"/>
 <wire x1="3.81" y1="2.54" x2="3.81" y2="6.35" width="1.016" layer="16" grouprefs="RNS"/>
+<wire x1="5.08" y1="29.21" x2="-1.27" y2="29.21" width="0.8128" layer="16"/>
+<wire x1="-1.27" y1="29.21" x2="-1.27" y2="6.35" width="0.8128" layer="16"/>
+<wire x1="-1.27" y1="6.35" x2="2.794" y2="6.35" width="0.8128" layer="16"/>
 <wire x1="3.81" y1="11.43" x2="5.08" y2="11.43" width="0" layer="19" extent="16-16"/>
 </signal>
@@
 <signal name="3.3V@2">
 <contactref element="U$1" pad="3.3V_2"/>
+<contactref element="JP6" pad="1"/>
+<wire x1="49.53" y1="57.15" x2="45.72" y2="57.15" width="0.8128" layer="16"/>
+<wire x1="45.72" y1="57.15" x2="43.18" y2="54.61" width="0.8128" layer="16"/>
+<wire x1="43.18" y1="54.61" x2="43.18" y2="53.34" width="0.8128" layer="16"/>
+<wire x1="43.18" y1="53.34" x2="33.02" y2="53.34" width="0.8128" layer="16"/>
 </signal>
 <signal name="GND@2">
 <contactref element="U$1" pad="GND_2"/>
 <contactref element="JP6" pad="2"/>
-<wire x1="49.53" y1="54.61" x2="41.91" y2="54.61" width="1.016" layer="16" grouprefs="RNS"/>
-<wire x1="41.91" y1="54.61" x2="40.64" y2="55.88" width="1.016" layer="16" grouprefs="RNS"/>
-<wire x1="40.64" y1="55.88" x2="33.02" y2="55.88" width="1.016" layer="16" grouprefs="RNS"/>
+<wire x1="33.02" y1="55.88" x2="41.91" y2="55.88" width="0.8128" layer="16"/>
+<wire x1="45.72" y1="59.69" x2="53.34" y2="59.69" width="0.8128" layer="16"/>
+<wire x1="53.34" y1="59.69" x2="53.34" y2="54.61" width="0.8128" layer="16"/>
+<wire x1="53.34" y1="54.61" x2="49.53" y2="54.61" width="0.8128" layer="16"/>
+<wire x1="41.91" y1="55.88" x2="45.72" y2="59.69" width="0.8128" layer="16"/>
 </signal>
 <signal name="GND@3">
