File: RNS_Board.sch (EAGLE design)
At the start: 6 parts

Commit message: Add files via upload
Connections:
- net 3.3V@2: now also JP6.1
- net 5V: no longer JP6.1
Changed lines of the file:
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@@
-</segment>
-<segment>
-<pinref part="JP6" gate="A" pin="1"/>
-<wire x1="149.86" y1="76.2" x2="137.16" y2="76.2" width="0.1524" layer="91" grouprefs="MPU_6050"/>
-<label x="139.7" y="76.2" size="1.778" layer="95" grouprefs="MPU_6050"/>
 </segment>
 <segment>
@@
 <label x="121.92" y="81.28" size="1.778" layer="95" align="bottom-right"/>
 </segment>
+<segment>
+<pinref part="JP6" gate="A" pin="1"/>
+<wire x1="149.86" y1="76.2" x2="137.16" y2="76.2" width="0.1524" layer="91" grouprefs="MPU_6050"/>
+<label x="139.7" y="76.2" size="1.778" layer="95" grouprefs="MPU_6050"/>
+</segment>
 </net>
